Commit message: actual URDF with mock LiDAR and platform assembly

File: base/base_description/urdf/_materials.urdf.xacro (robot description, xacro)
@@ -29,4 +29,7 @@
       <color rgba="0.1 0.1 0.1 1"/>
     </material>
+    <material name="green">
+      <color rgba="0.0 1.0 0.0 1"/>
+    </material>
  </xacro:unless>
 </robot>

File: base/base_description/urdf/_mockLiDAR.urdf.xacro (robot description, xacro)
@@ -1,4 +1,4 @@
 <?xml version="1.0"?>
-<robot xmlns:xacro="http://www.ros.org/wiki/xacro" name="basement_model">
+<robot xmlns:xacro="http://www.ros.org/wiki/xacro" name="lidar_model">
   <xacro:include filename="$(find base_description)/urdf/_materials.urdf.xacro"/>
   <!--
@@ -10,6 +10,6 @@
       scale   - control STL
   -->
-  <xacro:macro name="basement" params="parent
-              *origin name:=cheburashka
+  <xacro:macro name="ouster_lidar" params="parent
+              *origin name:=ouster
               scale:='1 1 1'">
       <!-- connection with parents -->
@@ -28,12 +28,12 @@
               <origin xyz="0.0 0.0 0.0" rpy="0.0 0.0 0.0"/>
               <geometry>
-                  <mesh filename="file://$(find base_description)/meshes/base-v3.stl" scale="${scale}" />
+                  <mesh filename="file://$(find base_description)/meshes/mockLiDAR.stl" scale="${scale}" />
               </geometry>
-              <material name="red"/>
+              <material name="green"/>
           </visual>
           <collision>
               <origin xyz="0.0 0.0 0.0" rpy="0.0 0.0 0.0"/>
               <geometry>
-                  <mesh filename="file://$(find base_description)/meshes/base-v3.stl" scale="${scale}" />
+                  <mesh filename="file://$(find base_description)/meshes/mockLiDAR.stl" scale="${scale}" />
               </geometry>
           </collision>
